Commit message: Added more joints

File: urdf/environment.xacro (robot description, xacro)
@@ -9,5 +9,5 @@
   <link name="world"/>
   <joint name="joint0" type="fixed">
-    <origin xyz="-0.65 0.0254 0" rpy="0 0 0"/>
+    <origin xyz="0.65 0.0254 0" rpy="0 0 0"/>
     <parent link="world"/>
     <child link="body"/>
@@ -38,5 +38,5 @@
     <parent link="body"/>
     <child link="nose"/>
-    <origin xyz="0 0 ${cyl_h + nose_r}" rpy="0 ${-PI/2} 0"/>
+    <origin xyz="0 0 ${cyl_h + nose_r}" rpy="0 ${PI/2} 0"/>
   </joint>
   <link name="nose">
@@ -66,5 +66,5 @@
     <parent link="body"/>
     <child link="test_tube"/>
-    <origin xyz="0.15 0 0" rpy="0 0 0"/>
+    <origin xyz="-0.15 0 0" rpy="0 0 0"/>
   </joint>
   <link name="test_tube">

Commit message: Added full translation control

File: urdf/environment.xacro (robot description, xacro)
@@ -9,5 +9,5 @@
   <link name="world"/>
   <joint name="joint0" type="fixed">
-    <origin xyz="0.65 0.0254 0" rpy="0 0 0"/>
+    <origin xyz="0.65 0.0508 0" rpy="0 0 0"/>
     <parent link="world"/>
     <child link="body"/>
@@ -66,5 +66,5 @@
     <parent link="body"/>
     <child link="test_tube"/>
-    <origin xyz="-0.15 0 0" rpy="0 0 0"/>
+    <origin xyz="-0.15 -0.0254 0" rpy="0 0 0"/>
   </joint>
   <link name="test_tube">

Commit message: Added different tube mesh

File: urdf/environment.xacro (robot description, xacro)
@@ -38,10 +38,12 @@
     <parent link="body"/>
     <child link="nose"/>
-    <origin xyz="0 0 ${cyl_h + nose_r}" rpy="0 ${PI/2} 0"/>
+    <origin xyz="0 0 ${cyl_h + nose_r}" rpy="0 ${PI/3} 0"/>
   </joint>
   <link name="nose">
     <collision>
+      <origin xyz="0 0 ${nose_h/2}" rpy="0 0 0"/>
       <geometry>
-        <mesh filename="model://hollow_tube/meshes/model.dae" scale="0.004 0.004 0.02"/>
+        <!--<mesh filename="model://hollow_tube/meshes/model.dae" scale="0.004 0.004 0.02"/>-->
+        <mesh filename="package://swab/meshes/cylinder.stl" scale="0.0016 0.0016 0.005"/>
         <!-- original outer diameter is 8.32 m -->
         <!-- original inner diameter is more than 3 m -->
@@ -49,6 +51,8 @@
     </collision>
     <visual>
+      <origin xyz="0 0 ${nose_h/2}" rpy="0 0 0"/>
       <geometry>
-        <mesh filename="model://hollow_tube/meshes/model.dae" scale="0.004 0.004 0.02"/>
+        <!--<mesh filename="model://hollow_tube/meshes/model.dae" scale="0.004 0.004 0.02"/>-->
+        <mesh filename="package://swab/meshes/cylinder.stl" scale="0.0016 0.0016 0.005"/>
         <!-- original outer diameter is 8.32 m -->
         <!-- original inner diameter is more than 3 m -->
@@ -70,6 +74,8 @@
   <link name="test_tube">
     <collision>
+      <origin xyz="0 0 ${nose_h/2}" rpy="0 0 0"/>
       <geometry>
-        <mesh filename="model://hollow_tube/meshes/model.dae" scale="0.004 0.004 0.02"/>
+        <!--<mesh filename="model://hollow_tube/meshes/model.dae" scale="0.004 0.004 0.02"/>-->
+        <mesh filename="package://swab/meshes/cylinder.stl" scale="0.0016 0.0016 0.005"/>
         <!-- original outer diameter is 8.32 m -->
         <!-- original inner diameter is more than 3 m -->
@@ -77,6 +83,8 @@
     </collision>
     <visual>
+      <origin xyz="0 0 ${nose_h/2}" rpy="0 0 0"/>
       <geometry>
-        <mesh filename="model://hollow_tube/meshes/model.dae" scale="0.004 0.004 0.02"/>
+        <!--<mesh filename="model://hollow_tube/meshes/model.dae" scale="0.004 0.004 0.02"/>-->
+        <mesh filename="package://swab/meshes/cylinder.stl" scale="0.0016 0.0016 0.005"/>
         <!-- original outer diameter is 8.32 m -->
         <!-- original inner diameter is more than 3 m -->

Commit message: Removed compliance since it wasn't meant to be on master yet

File: urdf/environment.xacro (robot description, xacro)
@@ -38,5 +38,5 @@
     <parent link="body"/>
     <child link="nose"/>
-    <origin xyz="0 0 ${cyl_h + nose_r}" rpy="0 ${PI/3} 0"/>
+    <origin xyz="0 0 ${cyl_h + nose_r}" rpy="0 ${PI/2} 0"/>
   </joint>
   <link name="nose">

Commit message: Environment cleanup

File: urdf/environment.xacro (robot description, xacro)
@@ -44,8 +44,5 @@
       <origin xyz="0 0 ${nose_h/2}" rpy="0 0 0"/>
       <geometry>
-        <!--<mesh filename="model://hollow_tube/meshes/model.dae" scale="0.004 0.004 0.02"/>-->
         <mesh filename="package://swab/meshes/cylinder.stl" scale="0.0016 0.0016 0.005"/>
-        <!-- original outer diameter is 8.32 m -->
-        <!-- original inner diameter is more than 3 m -->
       </geometry>
     </collision>
@@ -53,8 +50,5 @@
       <origin xyz="0 0 ${nose_h/2}" rpy="0 0 0"/>
       <geometry>
-        <!--<mesh filename="model://hollow_tube/meshes/model.dae" scale="0.004 0.004 0.02"/>-->
         <mesh filename="package://swab/meshes/cylinder.stl" scale="0.0016 0.0016 0.005"/>
-        <!-- original outer diameter is 8.32 m -->
-        <!-- original inner diameter is more than 3 m -->
       </geometry>
     </visual>
@@ -76,8 +70,5 @@
       <origin xyz="0 0 ${nose_h/2}" rpy="0 0 0"/>
       <geometry>
-        <!--<mesh filename="model://hollow_tube/meshes/model.dae" scale="0.004 0.004 0.02"/>-->
-        <mesh filename="package://swab/meshes/cylinder.stl" scale="0.0016 0.0016 0.005"/>
-        <!-- original outer diameter is 8.32 m -->
-        <!-- original inner diameter is more than 3 m -->
+        <mesh filename="package://swab/meshes/cylinder.stl" scale="0.0016 0.0016 0.004"/>
       </geometry>
     </collision>
@@ -85,8 +76,5 @@
       <origin xyz="0 0 ${nose_h/2}" rpy="0 0 0"/>
       <geometry>
-        <!--<mesh filename="model://hollow_tube/meshes/model.dae" scale="0.004 0.004 0.02"/>-->
-        <mesh filename="package://swab/meshes/cylinder.stl" scale="0.0016 0.0016 0.005"/>
-        <!-- original outer diameter is 8.32 m -->
-        <!-- original inner diameter is more than 3 m -->
+        <mesh filename="package://swab/meshes/cylinder.stl" scale="0.0016 0.0016 0.004"/>
       </geometry>
     </visual>

Commit message: Fixed compliance bugs. Pass-through still screws it up

File: urdf/environment.xacro (robot description, xacro)
@@ -35,4 +35,11 @@
     </inertial>
   </link>
+  <!--
+  <joint name="joint1" type="fixed">
+    <parent link="body"/>
+    <child link="nose"/>
+    <origin xyz="0 0 ${cyl_h + nose_r}" rpy="0 ${PI/2} ${PI/6}"/>
+  </joint>
+  -->
   <joint name="joint1" type="fixed">
     <parent link="body"/>
@@ -44,17 +51,11 @@
       <origin xyz="0 0 ${nose_h/2}" rpy="0 0 0"/>
       <geometry>
-        <!--<mesh filename="model://hollow_tube/meshes/model.dae" scale="0.004 0.004 0.02"/>-->
-        <mesh filename="package://swab/meshes/cylinder.stl" scale="0.0016 0.0016 0.005"/>
-        <!-- original outer diameter is 8.32 m -->
-        <!-- original inner diameter is more than 3 m -->
-      </geometry>
-    </collision>
-    <visual>
-      <origin xyz="0 0 ${nose_h/2}" rpy="0 0 0"/>
-      <geometry>
-        <!--<mesh filename="model://hollow_tube/meshes/model.dae" scale="0.004 0.004 0.02"/>-->
-        <mesh filename="package://swab/meshes/cylinder.stl" scale="0.0016 0.0016 0.005"/>
-        <!-- original outer diameter is 8.32 m -->
-        <!-- original inner diameter is more than 3 m -->
+        <mesh filename="package://swab/meshes/cylinder.stl" scale="0.0016 0.0016 0.005"/>
+      </geometry>
+    </collision>
+    <visual>
+      <origin xyz="0 0 ${nose_h/2}" rpy="0 0 0"/>
+      <geometry>
+        <mesh filename="package://swab/meshes/cylinder.stl" scale="0.0016 0.0016 0.005"/>
       </geometry>
     </visual>
@@ -67,4 +68,110 @@
     </inertial>
   </link>
+  <!--
+  <joint name="joint1" type="fixed">
+    <parent link="body"/>
+    <child link="nose_base"/>
+    <origin xyz="0 0 ${cyl_h}" rpy="0 0 ${PI/6}"/>
+  </joint>
+  <link name="nose_base">
+    <collision>
+      <origin xyz="0 0 0.005" rpy="0 0 0"/>
+      <geometry>
+        <box size="0.1 0.1 0.01"/>
+      </geometry>
+    </collision>
+    <visual>
+      <origin xyz="0 0 0.005" rpy="0 0 0"/>
+      <geometry>
+        <box size="0.1 0.1 0.01"/>
+      </geometry>
+    </visual>
+    <inertial>
+      <mass value="${mass}"/>
+      <inertia
+	  ixx="100" ixy="0.0" ixz="0.0"
+	  iyy="100" iyz="0.0"
+	  izz="100"/>
+    </inertial>
+  </link>
+  <joint name="joint_top" type="fixed">
+    <parent link="nose_base"/>
+    <child link="nose_top"/>
+    <origin xyz="0 0 0.02" rpy="0 0 0"/>
+  </joint>
+  <link name="nose_top">
+    <collision>
+      <origin xyz="0 0 0.005" rpy="0 0 0"/>
+      <geometry>
+        <box size="0.1 0.1 0.01"/>
+      </geometry>
+    </collision>
+    <visual>
+      <origin xyz="0 0 0.005" rpy="0 0 0"/>
+      <geometry>
+        <box size="0.1 0.1 0.01"/>
+      </geometry>
+    </visual>
+    <inertial>
+      <mass value="${mass}"/>
+      <inertia
+	  ixx="100" ixy="0.0" ixz="0.0"
+	  iyy="100" iyz="0.0"
+	  izz="100"/>
+    </inertial>
+  </link>
+  <joint name="joint_left" type="fixed">
+    <parent link="nose_base"/>
+    <child link="nose_left"/>
+    <origin xyz="0 -0.025 0.005" rpy="0 0 0"/>
+  </joint>
+  <link name="nose_left">
+    <collision>
+      <origin xyz="0 0 0.005" rpy="0 0 0"/>
+      <geometry>
+        <box size="0.1 0.01 0.02"/>
+      </geometry>
+    </collision>
+    <visual>
+      <origin xyz="0 0 0.005" rpy="0 0 0"/>
+      <geometry>
+        <box size="0.1 0.01 0.02"/>
+      </geometry>
+    </visual>
+    <inertial>
+      <mass value="${mass}"/>
+      <inertia
+	  ixx="100" ixy="0.0" ixz="0.0"
+	  iyy="100" iyz="0.0"
+	  izz="100"/>
+    </inertial>
+  </link>
+  <joint name="joint_right" type="fixed">
+    <parent link="nose_base"/>
+    <child link="nose_right"/>
+    <origin xyz="0 0.025 0.005" rpy="0 0 0"/>
+  </joint>
+  <link name="nose_right">
+    <collision>
+      <origin xyz="0 0 0.005" rpy="0 0 0"/>
+      <geometry>
+        <box size="0.1 0.01 0.02"/>
+      </geometry>
+    </collision>
+    <visual>
+      <origin xyz="0 0 0.005" rpy="0 0 0"/>
+      <geometry>
+        <box size="0.1 0.01 0.02"/>
+      </geometry>
+    </visual>
+    <inertial>
+      <mass value="${mass}"/>
+      <inertia
+	  ixx="100" ixy="0.0" ixz="0.0"
+	  iyy="100" iyz="0.0"
+	  izz="100"/>
+    </inertial>
+  </link>
+  -->
   <joint name="joint2" type="fixed">
     <parent link="body"/>
